File: JLink.kicad_sch (KiCad schematic)
At the start: 0 parts

Commit message: 2025/6/27：添加Lib ODBC库元器件
Parts:
- added U1: ~, IC:QFP50P1600X1600X160-100N, symbol libdb:IC/IC_001
Connections:
- new net: U1.10 (VSS), U1.27 (VSS), U1.74 (VSS)
- new net: U1.100 (VDD), U1.11 (VDD), U1.19 (VDD), U1.28 (VDD), U1.50 (VDD), U1.75 (VDD)

Commit message: 20250630
Parts:
- removed U1: ~, IC:QFP50P1600X1600X160-100N, symbol libdb:IC/IC_001
Other:
- added sheet Connect (Connect.kicad_sch)
- added sheet POWER (POWER.kicad_sch)
- added sheet STM32 (STM32.kicad_sch)
- added sheet USB (USB.kicad_sch)

Commit message: 基本完成
Other:
- sheet STM32 ports: added PDDM, PDDP; removed JTCK_SWCK, JTCK_SWDIO, JTDI, JTDO_SWO, JTRST
- sheet USB ports: added PDDM, PDDP; removed none
Changed lines of the file:
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@@
 	(generator_version "9.0")
 	(paper "A4")
+	(wire
+		(pts
+			(xy 123.19 139.7) (xy 127 139.7)
+		)
+		(stroke
+			(width 0)
+			(type default)
+		)
+	)
+	(wire
+		(pts
+			(xy 123.19 142.24) (xy 127 142.24)
+		)
+		(stroke
+			(width 0)
+			(type default)
+		)
+	)
 	(bus
 		(pts
@@
 		)
 	)
+	(wire
+		(pts
+			(xy 99.06 85.09) (xy 92.71 85.09)
+		)
+		(stroke
+			(width 0)
+			(type default)
+		)
+	)
+	(wire
+		(pts
+			(xy 99.06 82.55) (xy 92.71 82.55)
+		)
+		(stroke
+			(width 0)
+			(type default)
+		)
+	)
 	(bus
 		(pts
@@
 			(width 0)
 			(type default)
+		)
+	)
+	(label "PDDM"
+		(at 99.06 82.55 0)
+		(effects
+			(font
+				(size 1.27 1.27)
+			)
+			(justify left bottom)
 		)
 	)
@@
 		)
 	)
+	(label "PDDP"
+		(at 123.19 142.24 180)
+		(effects
+			(font
+				(size 1.27 1.27)
+			)
+			(justify right bottom)
+		)
+	)
 	(label "ADC[1..4]"
 		(at 123.19 59.69 0)
@@
 		)
 	)
+	(label "PDDM"
+		(at 123.19 139.7 180)
+		(effects
+			(font
+				(size 1.27 1.27)
+			)
+			(justify right bottom)
+		)
+	)
 	(label "PADC[1..4]"
 		(at 96.52 63.5 0)
+		(effects
+			(font
+				(size 1.27 1.27)
+			)
+			(justify left bottom)
+		)
+	)
+	(label "PDDP"
+		(at 99.06 85.09 0)
 		(effects
 			(font
@@
 			)
 		)
-		(pin "JTCK_SWCK" input
-			(at 92.71 48.26 0)
-			(effects
-				(font
-					(size 1.27 1.27)
-				)
-				(justify right)
-			)
-		)
-		(pin "JTCK_SWDIO" input
-			(at 92.71 50.8 0)
-			(effects
-				(font
-					(size 1.27 1.27)
-				)
-				(justify right)
-			)
-		)
-		(pin "JTDI" input
-			(at 92.71 53.34 0)
-			(effects
-				(font
-					(size 1.27 1.27)
-				)
-				(justify right)
-			)
-		)
-		(pin "JTDO_SWO" input
-			(at 92.71 55.88 0)
-			(effects
-				(font
-					(size 1.27 1.27)
-				)
-				(justify right)
-			)
-		)
-		(pin "JTRST" input
-			(at 92.71 58.42 0)
-			(effects
-				(font
-					(size 1.27 1.27)
-				)
-				(justify right)
-			)
-		)
 		(pin "NRST" output
 			(at 92.71 69.85 0)
@@
 		(pin "PADC[1..4]" bidirectional
 			(at 92.71 63.5 0)
+			(effects
+				(font
+					(size 1.27 1.27)
+				)
+				(justify right)
+			)
+		)
+		(pin "PDDM" input
+			(at 92.71 82.55 0)
+			(effects
+				(font
+					(size 1.27 1.27)
+				)
+				(justify right)
+			)
+		)
+		(pin "PDDP" input
+			(at 92.71 85.09 0)
 			(effects
 				(font
@@
 			)
 		)
+		(pin "PDDM" output
+			(at 127 139.7 180)
+			(effects
+				(font
+					(size 1.27 1.27)
+				)
+				(justify left)
+			)
+		)
+		(pin "PDDP" output
+			(at 127 142.24 180)
+			(effects
+				(font
+					(size 1.27 1.27)
+				)
+				(justify left)
+			)
+		)

Commit message: 修改内容中
Other:
- sheet STM32 ports: added PDDN; removed NRST, PDDM
- sheet USB ports: added PDDN; removed PDDM
Changed lines of the file:
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@@
 		)
 	)
-	(label "PDDM"
+	(label "PDDN"
 		(at 99.06 82.55 0)
 		(effects
@@
 		)
 	)
-	(label "PDDM"
+	(label "PDDN"
 		(at 123.19 139.7 180)
 		(effects
@@
 			)
 		)
-		(pin "NRST" output
-			(at 92.71 69.85 0)
-			(effects
-				(font
-					(size 1.27 1.27)
-				)
-				(justify right)
-			)
-		)
 		(pin "PADC[1..4]" bidirectional
 			(at 92.71 63.5 0)
@@
 			)
 		)
-		(pin "PDDM" input
-			(at 92.71 82.55 0)
-			(effects
-				(font
-					(size 1.27 1.27)
-				)
-				(justify right)
-			)
-		)
 		(pin "PDDP" input
 			(at 92.71 85.09 0)
+			(effects
+				(font
+					(size 1.27 1.27)
+				)
+				(justify right)
+			)
+		)
+		(pin "PDDN" input
+			(at 92.71 82.55 0)
 			(effects
 				(font
@@
 			)
 		)
-		(pin "PDDM" output
-			(at 127 139.7 180)
-			(effects
-				(font
-					(size 1.27 1.27)
-				)
-				(justify left)
-			)
-		)
 		(pin "PDDP" output
 			(at 127 142.24 180)
 			(effects
 				(font
+					(size 1.27 1.27)
+				)
+				(justify left)
+			)
+		)
+		(pin "PDDN" output
+			(at 127 139.7 180)
+			(effects
+				(font
