File: Connect.kicad_sch (KiCad schematic)
At the start: 44 parts

Commit message: JLINK will complite
Connections:
- net 3V3: now also RN3.6; no longer RN3.3
- net ENSRST: now also RN3.7; no longer RN3.2
- net P3V3: now also RN3.3; no longer RN3.7
- net P5V: now also RN3.4; no longer RN3.8
- net TIMA: now also Q2.2 (E), R7.2
- net TVRF: now also RN3.8; no longer RN3.1
- net VEE: now also RN3.2; no longer RN3.6
- net at Q2.1 (B), RN6.6: now also RN3.5; no longer RN3.4
- net at U7.3 (+INA), U7.5 (+INB): now also RN3.1; no longer RN3.5
- net at RN10.5: now also Q1.2, RN10.6; no longer U10.7 (B1)
- net at U10.6 (B2): now also RN10.7; no longer RN10.6
- new net: RN10.8, U10.7 (B1)
Changed lines of the file:
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@@
 		)
 	)
+	(label "TIMA"
+		(at 162.56 278.13 0)
+		(effects
+			(font
+				(size 1.27 1.27)
+			)
+			(justify left bottom)
+		)
+	)
 	(global_label "ETMS"
 		(shape input)
@@
 	)
 	(symbol
+		(lib_name "4D03WGJ0472T5E_1")
 		(lib_id "4D03WGJ0472T5E:4D03WGJ0472T5E")
 		(at 212.09 219.71 0)
+		(mirror y)
 		(unit 1)
 		(exclude_from_sim no)
@@
 		)
 		(property "Value" "10K"
-			(at 209.042 227.33 0)
+			(at 215.138 227.33 0)
 			(effects
 				(font
